Commit message: Fixes the helix length

File: urdf/copter_arm.urdf (robot description, URDF)
Before this commit: robot copter_arm, 3 links, 2 joints
Links:
- link helix: geometry collision box size=0.03 0.01 0.15; visual box size=0.03 0.001 0.30

Commit message: Making things lighter, and increasing speed limit of motor

File: urdf/copter_arm.urdf (robot description, URDF)
Before this commit: robot copter_arm, 3 links, 2 joints
Links:
- link arm: mass 0.1 -> 0.01
- link helix: mass 0.25 -> 0.1
Joints:
- joint motor_joint: limit effort=500 velocity=1100 -> effort=500 velocity=5000

Commit message: Initial import of the code needed for the real setup

File: urdf/copter_arm.urdf (robot description, URDF)
Before this commit: robot copter_arm, 3 links, 2 joints
Links:
- link arm: mass 0.01 -> 0.001; geometry collision box size=0.005 0.003 0.21; visual box size=0.005 0.003 0.21
- link helix: geometry collision box size=0.005 0.001 0.065; visual box size=0.005 0.001 0.065
Joints:
- joint motor_joint: limit effort=500 velocity=5000 -> effort=500 velocity=255; origin xyz=0 0.01 0.5 rpy=0 0 0 -> xyz=0 0.0015 0.21 rpy=0 0 0

Commit message: Changes reference to upward position.. also makes a nicer helix.

File: urdf/copter_arm.urdf (robot description, URDF)
Before this commit: robot copter_arm, 3 links, 2 joints
Links:
- link anchor: geometry collision box size=0.005 0.001 0.01; visual box size=0.005 0.001 0.01
- link helix: geometry collision box size=0.005 0.001 0.065; visual box size=0.005 0.001 0.065
Joints:
- joint free_joint: origin xyz=0 0 1.0 rpy=1.5708 0 0 -> xyz=0 0 1.0 rpy=0 0 0
- joint motor_joint: origin xyz=0 0.0015 0.21 rpy=0 0 0 -> xyz=0 0.01 0.21 rpy=0 0 0

Commit message: Makes reference to be rotated so zero means horizontal

File: urdf/copter_arm.urdf (robot description, URDF)
Before this commit: robot copter_arm, 3 links, 2 joints
Links:
- link helix: mass 0.1 -> 0.01
Joints:
- joint free_joint: origin xyz=0 0 1.0 rpy=0 0 0 -> xyz=0 0 1.0 rpy=${0.5*pi} 0 0
